File: 20180501 clock rgb.kicad_pcb (KiCad board)
At the start: 2 copper layers, 415 x 69 mm, 265 parts, among them J1 Barrel_Jack, J2 DB9M RS232, Q1 MMPQ2907A, Q2 MMPQ2907A, Q3 MMPQ2907A, SW1 SW_Push, SW2 SW_Push, SW3 SW_Push, SW4 SW_Push, SW5 SW_Push, SW6 SW_Push, U1 ATMEGA328P-PU, U2 74164, U3 74164, U4 LM358, U5 LM7805_TO220, U6 PCA8856B, U7 PCA8856B, U8 DS3231-8, U9 LM7812_TO220, Y1 16MHz

Commit message: Serial port work
Added MAX202 and supporting circuitry,
Changed LM358 to a SOIC package
Parts:
- added C10: 0.1uF, Capacitors_THT:CP_Radial_D5.0mm_P2.50mm, F.Cu at (302.3, 193.7)
- added C11: 0.1uF, Capacitors_THT:CP_Radial_D5.0mm_P2.50mm, F.Cu at (308.0, 192.4)
- added C12: 0.1uF, Capacitors_THT:CP_Radial_D5.0mm_P2.50mm, F.Cu at (297.8, 190.5)
- added C13: 0.1uF, Capacitors_THT:CP_Radial_D5.0mm_P2.50mm, F.Cu at (292.1, 188.0)
- added R132: 10k, Resistor_SMD:R_1210_3225Metric_Pad1.39x2.70mm_HandSolder, F.Cu at (323.2, 175.3)
- added R133: 10k, Resistor_SMD:R_1210_3225Metric_Pad1.39x2.70mm_HandSolder, F.Cu at (314.3, 192.4)
- added U10: MAX202, Housings_SOIC:SOIC-16_3.9x9.9mm_Pitch1.27mm, F.Cu at (306.7, 186.7)
- RN1: value 10K -> 10k; footprint Resistor_THT:R_Array_SIP8 -> Resistor_THT:R_Array_SIP4
- U4: footprint Package_DIP:DIP-8_W7.62mm -> Housings_SOIC:SOIC-8_3.9x4.9mm_Pitch1.27mm
- moved U4 22.9 mm to (276.9, 192.4), turned to 0 degrees
- moved RN1 19.1 mm to (322.6, 195.6), turned to 90 degrees
- moved R79 11.1 mm to (285.1, 189.9), turned to 135 degrees
- moved R80 10.5 mm to (286.4, 184.2), turned to 135 degrees
- moved D80 8.08 mm to (278.8, 186.1)
- moved D81 8.08 mm to (278.8, 179.7)
- moved R106 0.70 mm to (220.4, 220.6)
Connections:
- J2 pad 2: /RXD -> /TXD_PU
- J2 pad 3: /TXD -> Net-(J2-Pad3)
- J2 pad 4: /DTR -> /DTR_PU
- J2 pad 7: Net-(J2-Pad7) -> (no net)
- J2 pad 8: Net-(J2-Pad7) -> (no net)
- RN1 pad 2: /TXD -> /SCL
- RN1 pad 3: /RXD -> /SDA
- RN1 pad 4: /SCL -> /OE
- U1 pad 13: Net-(RN1-Pad8) -> (no net)
Routing:
- net Net-(R22-Pad1): track 305.9 -> 0.00 mm, vias 5 -> 0
- net Net-(RN1-Pad8): track 81.7 -> 0.00 mm
- net /RXD: track 78.2 -> 115.5 mm, vias 2 -> 10
- net /DTR: track 169.7 -> 138.8 mm, vias 1 -> 4
- net /TXD: track 88.6 -> 117.6 mm, vias 4 -> 11
- net +5V: track 162.0 -> 134.7 mm, vias 12 -> 10
- net /TXD_PU: track 0.00 -> 20.4 mm
- net /DTR_PU: track 0.00 -> 17.9 mm, vias 0 -> 1
- net Net-(C13-Pad2): track 0.00 -> 16.0 mm
- net Earth: track 81.5 -> 95.1 mm, vias 11 -> 14
- net Net-(R79-Pad1): track 4.83 -> 15.6 mm
- net /SCL: track 294.2 -> 303.5 mm, vias 9 -> 11
- net Net-(C12-Pad1): track 0.00 -> 7.83 mm
- net Net-(C9-Pad2): track 101.2 -> 107.3 mm
- net Net-(C11-Pad2): track 0.00 -> 5.89 mm
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