File: 20180501 clock rgb.sch (KiCad schematic (older format))
At the start: 265 parts, among them J1 Barrel_Jack, J2 DB9M RS232, Q1 MMPQ2907A, Q2 MMPQ2907A, Q3 MMPQ2907A, SW1 SW_Push, SW2 SW_Push, SW3 SW_Push, SW4 SW_Push, SW5 SW_Push, SW6 SW_Push, U1 ATMEGA328P-PU, U2 74164, U3 74164, U4 LM358, U5 LM7805_TO220, U6 PCA8856B, U7 PCA8856B, U8 DS3231-8, U9 LM7812_TO220, Y1 16MHz

Commit message: Serial port work
Added MAX202 and supporting circuitry,
Changed LM358 to a SOIC package
Parts:
- removed RN1: 10K, Resistor_THT:R_Array_SIP8, symbol R_Network07
- added C10, C11, C12, C13: 0.1uF, Capacitors_THT:CP_Radial_D5.0mm_P2.50mm, symbol CP
- added R132, R133: 10k, Resistor_SMD:R_1210_3225Metric_Pad1.39x2.70mm_HandSolder, symbol R
- added RN1: 10k, Resistor_THT:R_Array_SIP4, symbol R_Network03
- added U10: MAX202, Housings_SOIC:SOIC-16_3.9x9.9mm_Pitch1.27mm, symbol MAX202
- C6, C8, C9: symbol C -> CP
- U4: footprint Package_DIP:DIP-8_W7.62mm -> Housings_SOIC:SOIC-8_3.9x4.9mm_Pitch1.27mm
Connections:
- net +5V: now also RN1.1 (common), U10.16 (VCC)
- net DTR: now also U10.9 (R2OUT); no longer J2.4
- net Earth: now also C12.2, C13.1, R132.1, R133.1, U10.15 (GND)
- net OE: now also RN1.4 (R3)
- net RXD: now also U10.11 (T1IN); no longer J2.2
- net SCL: now also RN1.2 (R1)
- net SDA: now also RN1.3 (R2)
- net TXD: now also U10.12 (R1OUT); no longer J2.3
- net at J2.7: no longer J2.8
- new net: C10.1, U10.1 (C1+)
- new net: J2.3, U10.14 (T1OUT)
- new net: C12.1, U10.2 (VS+)
- new net: C10.2, U10.3 (C1-)
- new net: C11.1, U10.4 (C2+)
- new net: C11.2, U10.5 (C2-)
- new net: C13.2, U10.6 (VS-)
- new net DTR_PU: J2.4, R133.2, U10.8 (R2IN)
- new net TXD_PU: J2.2, R132.2, U10.13 (R1IN)
- no-connect marks 17 -> 22
Other:
- note added: "TX/RX relative to PC"

Commit message: created gerber files
final, ready to send in to jlcpcb
Parts:
- removed U4: LM358, Housings_SOIC:SOIC-8_3.9x4.9mm_Pitch1.27mm, symbol LM358
Connections:
- net +5V: now also U2.14 (Vdd), U3.14 (Vdd)
- net Earth: now also U2.7 (Vss), U3.7 (Vss)
- net RXD: now also R80.1
- net TXD: now also R79.1
