File: bak.kicad_pcb (KiCad board)
At the start: 2 copper layers, 415 x 69 mm, 275 parts, among them J1 Barrel_Jack, J2 DB9M RS232, Q1 MMPQ2907A, Q2 MMPQ2907A, Q3 MMPQ2907A, SW1 SW_Push, SW2 SW_Push, SW3 SW_Push, SW4 SW_Push, SW5 SW_Push, SW6 SW_Push, U1 ATMEGA328P-PU, U10 MAX202, U2 74164, U3 74164, U5 LM7805_TO220, U6 PCA8856B, U7 PCA8856B, U8 DS3231-8, U9 LM7812_TO220, Y1 16MHz

Commit message: created gerber files
final, ready to send in to jlcpcb
Parts:
- moved R103 0.50 mm to (223.1, 210.4)
- moved R106 0.40 mm to (220.4, 220.6)
- moved R92 0.25 mm to (323.0, 217.2)
- moved R104 0.23 mm to (265.0, 181.5)
Routing:
- net Net-(RV4-Pad2): track 162.9 -> 0.00 mm
- net Earth: track 223.8 -> 92.4 mm, vias 15 -> 12
- net +5V: track 285.5 -> 222.7 mm, vias 17 -> 12
- net Net-(D45-Pad1): track 657.2 -> 636.1 mm
- net /OE: track 279.3 -> 278.2 mm
- net Net-(C9-Pad2): track 109.0 -> 108.0 mm
