File: _saved_20180501 clock rgb.sch (KiCad schematic (older format))
At the start: 271 parts, among them J1 Barrel_Jack, J2 DB9M RS232, Q1 MMPQ2907A, Q2 MMPQ2907A, Q3 MMPQ2907A, SW1 SW_Push, SW2 SW_Push, SW3 SW_Push, SW4 SW_Push, SW5 SW_Push, SW6 SW_Push, U1 ATMEGA328P-PU, U10 MAX202, U2 74164, U3 74164, U5 LM7805_TO220, U6 PCA8856B, U7 PCA8856B, U8 DS3231-8, U9 LM7812_TO220, Y1 16MHz

Commit message: jesus github
asdf
Parts:
- D14, D21: value LED_ARGB -> APFA3010
- D22, D23, D24, D25, D26, D27, D28, D29, D30, D31, D32, D33, D34, D35, D36, D37, D38, D39, D40, D41, D42, D43, D44, D45, D46, D47, D48, D49, D50, D51, D52, D53, D54, D55, D56, D57, D58, D59, D60, D61, D62, D63, D64, D65, D66, D67, D68, D69, D70, D71, D72, D73, D74, D75, D76, D77, D78, D79, D82, D83, D84, D85, D86, D87, D88, D91, D92, D93, D94, D95, D96, D97: symbol LED_ARGB -> APFA3010
Connections:
- net +12V: now also D43.2 (A), D44.2 (A); no longer D43.1 (A), D44.1 (A)
- net R: now also D22.1 (R), D23.1 (R), D24.1 (R), D25.1 (R), D26.1 (R), D27.1 (R), D28.1 (R), D29.1 (R), D30.1 (R), D31.1 (R), D32.1 (R), D33.1 (R), D34.1 (R), D35.1 (R), D36.1 (R), D37.1 (R), D38.1 (R), D39.1 (R), D40.1 (R), D41.1 (R), D42.1 (R), D43.1 (R), D44.1 (R), D45.1 (R), D46.1 (R), D47.1 (R), D48.1 (R), D49.1 (R), D50.1 (R), D51.1 (R), D52.1 (R), D53.1 (R), D54.1 (R), D55.1 (R), D56.1 (R), D57.1 (R), D58.1 (R), D59.1 (R), D60.1 (R), D61.1 (R), D62.1 (R), D63.1 (R), D64.1 (R), D65.1 (R), D66.1 (R), D67.1 (R), D68.1 (R), D69.1 (R), D70.1 (R), D71.1 (R), D72.1 (R), D73.1 (R), D74.1 (R), D75.1 (R), D76.1 (R), D77.1 (R), D78.1 (R), D79.1 (R), D82.1 (R), D83.1 (R), D84.1 (R), D85.1 (R), D86.1 (R), D87.1 (R), D88.1 (R); no longer D22.2 (RK), D23.2 (RK), D24.2 (RK), D25.2 (RK), D26.2 (RK), D27.2 (RK), D28.2 (RK), D29.2 (RK), D30.2 (RK), D31.2 (RK), D32.2 (RK), D33.2 (RK), D34.2 (RK), D35.2 (RK), D36.2 (RK), D37.2 (RK), D38.2 (RK), D39.2 (RK), D40.2 (RK), D41.2 (RK), D42.2 (RK), D43.2 (RK), D44.2 (RK), D45.2 (RK), D46.2 (RK), D47.2 (RK), D48.2 (RK), D49.2 (RK), D50.2 (RK), D51.2 (RK), D52.2 (RK), D53.2 (RK), D54.2 (RK), D55.2 (RK), D56.2 (RK), D57.2 (RK), D58.2 (RK), D59.2 (RK), D60.2 (RK), D61.2 (RK), D62.2 (RK), D63.2 (RK), D64.2 (RK), D65.2 (RK), D66.2 (RK), D67.2 (RK), D68.2 (RK), D69.2 (RK), D70.2 (RK), D71.2 (RK), D72.2 (RK), D73.2 (RK), D74.2 (RK), D75.2 (RK), D76.2 (RK), D77.2 (RK), D78.2 (RK), D79.2 (RK), D82.2 (RK), D83.2 (RK), D84.2 (RK), D85.2 (RK), D86.2 (RK), D87.2 (RK), D88.2 (RK)
- net at Q2.3 (C2), Q2.4 (C2): now also D91.2 (A); no longer D91.1 (A)
- net at Q2.5 (C3), Q2.6 (C3): now also D92.2 (A); no longer D92.1 (A)
- net at Q2.7 (C4), Q2.8 (C4): now also D93.2 (A); no longer D93.1 (A)
- net at R111.1: now also D91.1 (R); no longer D91.2 (RK)
- net at R114.1: now also D92.1 (R); no longer D92.2 (RK)
- net at R117.1: now also D93.1 (R); no longer D93.2 (RK)
- net at Q3.1 (C1), Q3.2 (C1): now also D94.2 (A); no longer D94.1 (A)
- net at R120.1: now also D94.1 (R); no longer D94.2 (RK)
- net at Q3.3 (C2), Q3.4 (C2): now also D95.2 (A); no longer D95.1 (A)
- net at R123.1: now also D95.1 (R); no longer D95.2 (RK)
- net at Q3.5 (C3), Q3.6 (C3): now also D96.2 (A); no longer D96.1 (A)
- net at R126.1: now also D96.1 (R); no longer D96.2 (RK)
- net at Q3.7 (C4), Q3.8 (C4): now also D97.2 (A); no longer D97.1 (A)
- net at R129.1: now also D97.1 (R); no longer D97.2 (RK)
- new net: D22.2 (A), D23.2 (A), D24.2 (A), D25.2 (A), D26.2 (A), D27.2 (A), D28.2 (A), D29.2 (A), D30.2 (A), D31.2 (A), D32.2 (A), D33.2 (A), D34.2 (A), D35.2 (A), D36.2 (A), D37.2 (A), D38.2 (A), D39.2 (A), D40.2 (A), D41.2 (A), D42.2 (A), Q1.3 (C2), Q1.4 (C2)
- new net: D45.2 (A), D46.2 (A), D47.2 (A), D48.2 (A), D49.2 (A), D50.2 (A), D51.2 (A), D52.2 (A), D53.2 (A), D54.2 (A), D55.2 (A), D56.2 (A), D57.2 (A), D58.2 (A), D59.2 (A), D60.2 (A), D61.2 (A), D62.2 (A), D63.2 (A), D64.2 (A), D65.2 (A), Q1.5 (C3), Q1.6 (C3)
- new net: D66.2 (A), D67.2 (A), D68.2 (A), D69.2 (A), D70.2 (A), D71.2 (A), D72.2 (A), D73.2 (A), D74.2 (A), D75.2 (A), D76.2 (A), D77.2 (A), D78.2 (A), D79.2 (A), D82.2 (A), D83.2 (A), D84.2 (A), D85.2 (A), D86.2 (A), D87.2 (A), D88.2 (A), Q1.7 (C4), Q1.8 (C4)
